File: tannenbaum.kicad_sch (KiCad schematic)
At the start: 0 parts

Commit message: sym
Parts:
- added C1: 100n, symbol Device:C
- added C2: 100p, symbol Device:C
- added C3: 22u, symbol Device:C
- added D1, D10, D11, D12, D2, D3, D4, D5, D6, D7, D8, D9: LED, symbol Device:LED
- added D13: 1N4148W, Diode_SMD:D_SOD-123, symbol Diode:1N4148W
- added Q1: 2N7002, digikey-footprints:SOT-23-3, symbol dk_Transistors-FETs-MOSFETs-Single:2N7002
- added Q2, Q3, Q4, Q5: MMBT3904-7-F, digikey-footprints:SOT-23-3, symbol dk_Transistors-Bipolar-BJT-Single:MMBT3904-7-F
- added R1, R2, R3, R4: 1K2, symbol Device:R
- added R10, R11, R12, R9: R_Trim, symbol Device:R_Trim
- added R5, R6, R7, R8: 100k, symbol Device:R
- added U1: ICM7555IPAZ, digikey-footprints:DIP-8_W7.62mm, symbol dk_Clock-Timing-Programmable-Timers-and-Oscillators:ICM7555IPAZ

Commit message: sym
Parts:
- C1: footprint (none) -> Capacitor_SMD:C_0805_2012Metric
- C2: footprint (none) -> Capacitor_SMD:C_0603_1608Metric
- C3: footprint (none) -> Capacitor_SMD:CP_Elec_6.3x5.7
- D1: renamed from D2; footprint (none) -> LED_SMD:LED_0805_2012Metric
- D10: renamed from D8; footprint (none) -> LED_SMD:LED_0805_2012Metric
- D11, D3: footprint (none) -> LED_SMD:LED_0805_2012Metric
- D12: renamed from D5; footprint (none) -> LED_SMD:LED_0805_2012Metric
- D2: renamed from D9; footprint (none) -> LED_SMD:LED_0805_2012Metric
- D4: renamed from D12; footprint (none) -> LED_SMD:LED_0805_2012Metric
- D5: renamed from D1; footprint (none) -> LED_SMD:LED_0805_2012Metric
- D6: renamed from D10; footprint (none) -> LED_SMD:LED_0805_2012Metric
- D7: renamed from D6; footprint (none) -> LED_SMD:LED_0805_2012Metric
- D8: renamed from D4; footprint (none) -> LED_SMD:LED_0805_2012Metric
- D9: renamed from D7; footprint (none) -> LED_SMD:LED_0805_2012Metric
- R1: renamed from R3; footprint (none) -> Resistor_SMD:R_0603_1608Metric
- R10: renamed from R7; footprint (none) -> Resistor_SMD:R_0805_2012Metric
- R11: renamed from R5; footprint (none) -> Resistor_SMD:R_0805_2012Metric
- R12: renamed from R6; footprint (none) -> Resistor_SMD:R_0805_2012Metric
- R2: renamed from R1; footprint (none) -> Resistor_SMD:R_0603_1608Metric
- R3: renamed from R2; footprint (none) -> Resistor_SMD:R_0603_1608Metric
- R4: footprint (none) -> Resistor_SMD:R_0603_1608Metric
- R5: renamed from R12; footprint (none) -> PVG5A202C03R00:TRIM_PVG5A202C03R00
- R6: renamed from R11; footprint (none) -> PVG5A202C03R00:TRIM_PVG5A202C03R00
- R7: renamed from R10; footprint (none) -> PVG5A202C03R00:TRIM_PVG5A202C03R00
- R8: renamed from R9; footprint (none) -> PVG5A202C03R00:TRIM_PVG5A202C03R00
- R9: renamed from R8; footprint (none) -> Resistor_SMD:R_0805_2012Metric
- renumbered Q5 to Q1, Q3 to Q2, Q2 to Q3, Q1 to Q5
Other:
- moved on the sheet: C1, C2, C3, D1, D10, D11, D12, D2, D3, D4, D5, D6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

Commit message: predr
Connections:
- net GND: now reaches C1.1
- net GND: now also C2.2, C3.2, Q5.2 (S), R5.2, R6.2, R7.2, R8.2, U1.1 (GND)
- net 3V3: now reaches C1.2
- net 3V3: now also R11.2, R9.1, U1.4 (~{RESET}), U1.8 (VDD)
- net at R2.1: now also Q3.2 (E)
- net at R2.2: now also R7.1
- net at R12.1: now also U1.3 (OUT)
- net CMD: now reaches R12.2
- net CMD: now also Q1.1 (B), Q2.1 (B), Q5.1 (G)
- net BLU_ON: now reaches R9.2
- net BLU_ON: now also Q3.1 (B), Q4.1 (B), Q5.3 (D)
- net at D10.1 (K): now also Q2.3 (C)
- net at D10.2 (A): now also D6.1 (K)
- net at R4.1: now also Q1.2 (E)
- net at R4.2: now also R5.1
- net at D7.1 (K): now also D11.2 (A)
- net at D7.2 (A): now also D3.1 (K)
- net at R6.1: now also R1.2
- net at D11.1 (K): now also Q3.3 (C)
- net at R3.1: now also Q4.2 (E)
- net at R3.2: now also R8.1
- net at D12.1 (K): now also Q4.3 (C)
- net at D12.2 (A): now also D8.1 (K)
- net DSC: now reaches R10.1
- net DSC: now also D13.2 (A), R11.1, U1.7 (DISCH)
- net THR: now reaches R10.2
- net THR: now also C3.1, D13.1 (K), U1.2 (~{TRIG}), U1.6 (THRES)
- net at D2.1 (K): now also D6.2 (A)
- net 9V: now reaches D2.2 (A)
- net 9V: now also D1.2 (A), D3.2 (A), D4.2 (A)
- net at Q1.3 (C): now also D9.1 (K)
- net at D9.2 (A): now also D5.1 (K)
- net at C2.1: now also U1.5 (CONT)
- net at D4.1 (K): now also D8.2 (A)
- net at Q2.2 (E): now also R1.1
- net at D5.2 (A): now also D1.1 (K)
Other:
- sheet PSU ports: added 3V3, 9V; removed none
- note added: "BLU"
- note added: "VERDE"
- moved on the sheet: C1, C2, C3, D1, D10, D13, D2, D3, D4, D5, D6, D7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

Commit message: predr
Parts:
- Q1: Purpose (none) -> C.C. driver
- Q2, Q3, Q4: Purpose (none) -> C. C. driver
- Q5: Purpose (none) -> Inverting Switch
- U1: Purpose (none) -> Astable Multivibrator
Connections:
- net CV2: now reaches D10.1 (K), Q2.3 (C)
- net CB1: now reaches D11.1 (K), Q3.3 (C)
- net CB2: now reaches D12.1 (K), Q4.3 (C)
- net CV1: now reaches D9.1 (K), Q1.3 (C)
Other:
- moved on the sheet: D10, D11, D12, D9
Changed lines of the file:
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@@
     (stroke (width 0) (type default))
   )
-  (wire (pts (xy 138.43 58.42) (xy 138.43 60.96))
+  (wire (pts (xy 138.43 54.61) (xy 138.43 60.96))
     (stroke (width 0) (type default))
   )
@@
     (stroke (width 0) (type default))
   )
-  (wire (pts (xy 231.14 44.45) (xy 231.14 50.8))
+  (wire (pts (xy 231.14 44.45) (xy 231.14 46.99))
     (stroke (width 0) (type default))
   )
@@
     (stroke (width 0) (type default))
   )
-  (wire (pts (xy 138.43 43.18) (xy 138.43 50.8))
-    (stroke (width 0) (type default))
-  )
-  (wire (pts (xy 256.54 58.42) (xy 256.54 60.96))
-    (stroke (width 0) (type default))
-  )
-  (wire (pts (xy 231.14 58.42) (xy 231.14 60.96))
+  (wire (pts (xy 138.43 43.18) (xy 138.43 46.99))
+    (stroke (width 0) (type default))
+  )
+  (wire (pts (xy 256.54 54.61) (xy 256.54 60.96))
+    (stroke (width 0) (type default))
+  )
+  (wire (pts (xy 231.14 54.61) (xy 231.14 60.96))
     (stroke (width 0) (type default))
   )
@@
     (stroke (width 0) (type default))
   )
-  (wire (pts (xy 161.29 58.42) (xy 161.29 60.96))
+  (wire (pts (xy 161.29 54.61) (xy 161.29 60.96))
     (stroke (width 0) (type default))
   )
@@
     (stroke (width 0) (type default))
   )
-  (wire (pts (xy 161.29 44.45) (xy 161.29 50.8))
+  (wire (pts (xy 161.29 44.45) (xy 161.29 46.99))
     (stroke (width 0) (type default))
   )
@@
     (stroke (width 0) (type default))
   )
-  (wire (pts (xy 256.54 44.45) (xy 256.54 50.8))
+  (wire (pts (xy 256.54 44.45) (xy 256.54 46.99))
     (stroke (width 0) (type default))
   )
@@
     (effects (font (size 1.27 1.27)) (justify left bottom))
   )
+  (label "CB2" (at 256.54 59.69 0) (fields_autoplaced)
+    (effects (font (size 1.27 1.27)) (justify left bottom))
+  )
   (label "CMD" (at 139.7 119.38 0) (fields_autoplaced)
     (effects (font (size 1.27 1.27)) (justify left bottom))
   )
+  (label "CB1" (at 231.14 59.69 0) (fields_autoplaced)
+    (effects (font (size 1.27 1.27)) (justify left bottom))
+  )
   (label "3V3" (at 198.12 78.74 0) (fields_autoplaced)
     (effects (font (size 1.27 1.27)) (justify left bottom))
@@
   )
   (label "3V3" (at 109.22 110.49 90) (fields_autoplaced)
+    (effects (font (size 1.27 1.27)) (justify left bottom))
+  )
+  (label "CV2" (at 161.29 59.69 0) (fields_autoplaced)
+    (effects (font (size 1.27 1.27)) (justify left bottom))
+  )
+  (label "CV1" (at 138.43 59.69 0) (fields_autoplaced)
     (effects (font (size 1.27 1.27)) (justify left bottom))
   )
@@
     )
   )
-  (symbol (lib_id "Device:LED") (at 161.29 54.61 90) (unit 1)
-    (in_bom yes) (on_board yes) (dnp no) (fields_autoplaced)
-    (property "Reference" "D10" (at 154.94 56.1975 0)
-      (effects (font (size 1.27 1.27)))
-    )
-    (property "Value" "LED" (at 157.48 56.1975 0)
-      (effects (font (size 1.27 1.27)))
-    )
-    (property "Footprint" "LED_SMD:LED_0805_2012Metric" (at 161.29 54.61 0)
-      (effects (font (size 1.27 1.27)) hide)
-    )
-    (property "Datasheet" "~" (at 161.29 54.61 0)
+  (symbol (lib_id "Device:LED") (at 161.29 50.8 90) (unit 1)
+    (in_bom yes) (on_board yes) (dnp no) (fields_autoplaced)
+    (property "Reference" "D10" (at 154.94 52.3875 0)
+      (effects (font (size 1.27 1.27)))
+    )
+    (property "Value" "LED" (at 157.48 52.3875 0)
+      (effects (font (size 1.27 1.27)))
+    )
+    (property "Footprint" "LED_SMD:LED_0805_2012Metric" (at 161.29 50.8 0)
+      (effects (font (size 1.27 1.27)) hide)
+    )
+    (property "Datasheet" "~" (at 161.29 50.8 0)
       (effects (font (size 1.27 1.27)) hide)
     )
@@
     )
   )
-  (symbol (lib_id "Device:LED") (at 231.14 54.61 90) (unit 1)
-    (in_bom yes) (on_board yes) (dnp no) (fields_autoplaced)
-    (property "Reference" "D11" (at 224.79 56.1975 0)
-      (effects (font (size 1.27 1.27)))
-    )
-    (property "Value" "LED" (at 227.33 56.1975 0)
-      (effects (font (size 1.27 1.27)))
-    )
-    (property "Footprint" "LED_SMD:LED_0805_2012Metric" (at 231.14 54.61 0)
-      (effects (font (size 1.27 1.27)) hide)
-    )
-    (property "Datasheet" "~" (at 231.14 54.61 0)
+  (symbol (lib_id "Device:LED") (at 231.14 50.8 90) (unit 1)
+    (in_bom yes) (on_board yes) (dnp no) (fields_autoplaced)
+    (property "Reference" "D11" (at 224.79 52.3875 0)
+      (effects (font (size 1.27 1.27)))
+    )
+    (property "Value" "LED" (at 227.33 52.3875 0)
+      (effects (font (size 1.27 1.27)))
+    )
+    (property "Footprint" "LED_SMD:LED_0805_2012Metric" (at 231.14 50.8 0)
+      (effects (font (size 1.27 1.27)) hide)
+    )
+    (property "Datasheet" "~" (at 231.14 50.8 0)
       (effects (font (size 1.27 1.27)) hide)
     )
@@
   )
   (symbol (lib_id "dk_Transistors-FETs-MOSFETs-Single:2N7002") (at 198.12 116.84 0) (unit 1)
-    (in_bom yes) (on_board yes) (dnp no) (fields_autoplaced)
+    (in_bom yes) (on_board yes) (dnp no)
     (property "Reference" "Q5" (at 201.93 115.57 0)
       (effects (font (size 1.524 1.524)) (justify left))
@@
       (effects (font (size 1.524 1.524)) (justify left) hide)
     )
+    (property "Purpose" "Inverting Switch" (at 187.96 123.19 0)
+      (effects (font (size 1.27 1.27)))
+    )
     (pin "1")
     (pin "2")
@@
     )
   )
-  (symbol (lib_id "Device:LED") (at 256.54 54.61 90) (unit 1)
-    (in_bom yes) (on_board yes) (dnp no) (fields_autoplaced)
-    (property "Reference" "D12" (at 250.19 56.1975 0)
-      (effects (font (size 1.27 1.27)))
-    )
-    (property "Value" "LED" (at 252.73 56.1975 0)
-      (effects (font (size 1.27 1.27)))
-    )
-    (property "Footprint" "LED_SMD:LED_0805_2012Metric" (at 256.54 54.61 0)
-      (effects (font (size 1.27 1.27)) hide)
-    )
-    (property "Datasheet" "~" (at 256.54 54.61 0)
+  (symbol (lib_id "Device:LED") (at 256.54 50.8 90) (unit 1)
+    (in_bom yes) (on_board yes) (dnp no) (fields_autoplaced)
+    (property "Reference" "D12" (at 250.19 52.3875 0)
+      (effects (font (size 1.27 1.27)))
+    )
+    (property "Value" "LED" (at 252.73 52.3875 0)
+      (effects (font (size 1.27 1.27)))
+    )
+    (property "Footprint" "LED_SMD:LED_0805_2012Metric" (at 256.54 50.8 0)
+      (effects (font (size 1.27 1.27)) hide)
+    )
+    (property "Datasheet" "~" (at 256.54 50.8 0)
       (effects (font (size 1.27 1.27)) hide)
     )
@@
       (effects (font (size 1.524 1.524)) (justify left) hide)
     )
+    (property "Purpose" "C.C. driver" (at 121.92 63.5 0)
+      (effects (font (size 1.27 1.27)) (justify left bottom))
+    )
     (pin "1")
     (pin "2")
@@
     )
   )
-  (symbol (lib_id "Device:LED") (at 138.43 54.61 90) (unit 1)
+  (symbol (lib_id "Device:LED") (at 138.43 50.8 90) (unit 1)
     (in_bom yes) (on_board yes) (dnp no)
-    (property "Reference" "D9" (at 131.3025 56.2467 0)
-      (effects (font (size 1.27 1.27)))
-    )
-    (property "Value" "LED" (at 134.62 56.1975 0)
-      (effects (font (size 1.27 1.27)))
-    )
-    (property "Footprint" "LED_SMD:LED_0805_2012Metric" (at 138.43 54.61 0)
-      (effects (font (size 1.27 1.27)) hide)
-    )
-    (property "Datasheet" "~" (at 138.43 54.61 0)
+    (property "Reference" "D9" (at 131.3025 52.4367 0)
+      (effects (font (size 1.27 1.27)))
+    )
+    (property "Value" "LED" (at 134.62 52.3875 0)
+      (effects (font (size 1.27 1.27)))
+    )
+    (property "Footprint" "LED_SMD:LED_0805_2012Metric" (at 138.43 50.8 0)
+      (effects (font (size 1.27 1.27)) hide)
+    )
+    (property "Datasheet" "~" (at 138.43 50.8 0)
       (effects (font (size 1.27 1.27)) hide)
     )
@@
       (effects (font (size 1.524 1.524)) (justify left) hide)
     )
+    (property "Purpose" "C. C. driver" (at 246.38 62.23 0)
+      (effects (font (size 1.27 1.27)))
+    )
     (pin "1")
     (pin "2")
@@
       (effects (font (size 1.524 1.524)) (justify left) hide)
     )
+    (property "Purpose" "C. C. driver" (at 147.32 60.96 0)
+      (effects (font (size 1.27 1.27)) (justify left top))
+    )
     (pin "1")
     (pin "2")
@@
       (effects (font (size 1.524 1.524)) (justify left) hide)
     )
+    (property "Purpose" "C. C. driver" (at 222.25 62.23 0)
+      (effects (font (size 1.27 1.27)))
+    )
     (pin "1")
     (pin "2")
@@
       (effects (font (size 1.524 1.524)) (justify left) hide)
     )
-    (pin "1")
+    (property "Purpose" "Astable Multivibrator" (at 93.98 105.41 0)
+      (effects (font (size 1.27 1.27)))
+    )
+    (pin "1")

Commit message: predr
Parts:
- D1: Purpose (none) -> L1 Verde 1
- D10: Purpose (none) -> L3 Verde 2
- D11: Purpose (none) -> L3 Blu 1
- D12: Purpose (none) -> L3 Blu 2
- D2: Purpose (none) -> L1 Verde 2
- D3: Purpose (none) -> L1 Blu 1
- D4: Purpose (none) -> L1 Blu 2
- D5: Purpose (none) -> L2 Verde 1
- D6: Purpose (none) -> L2 Verde 2
- D7: Purpose (none) -> L2 Blu 1
- D8: Purpose (none) -> L2 Blu 2
- D9: Purpose (none) -> L3 Verde 1
- R1: Purpose (none) -> RV2
- R2: Purpose (none) -> RB1
- R3: Purpose (none) -> RB2
- R4: Purpose (none) -> RV1
- R5: Purpose (none) -> TV1
- R6: Purpose (none) -> TV2
- R7: Purpose (none) -> TB1
- R8: Purpose (none) -> TB2
Other:
- moved on the sheet: D5, D6, D7, D8

Commit message: gitignore e revised sch
Connections:
- net BLU_ON renamed /CMD
Other:
- note added: "Clock CMD"
- note added: "Inverter"
- moved on the sheet: C1, C2, C3, D1, D10, D13, D2, D5, D6, D9, Q1, Q2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
