File: tannenbaum.kicad_pcb (KiCad board)
At the start: 2 copper layers, 41 parts, among them Q1 MMBT3904-7-F, Q2 MMBT3904-7-F, Q3 MMBT3904-7-F, Q4 MMBT3904-7-F, Q5 2N7002, Q6 BSS84, SW1 SW_SPDT, U1 ICM7555IPAZ, U2 AP7380-33Y-13

Commit message: pcb
Parts:
- added C6: 10n, Capacitor_SMD:C_0805_2012Metric, F.Cu at (1.73, 5.46)
- added U2: LP2985-3.3, Package_TO_SOT_SMD:SOT-23-5, F.Cu at (2.08, 1.73)
- moved BT1 526.6 mm to (44.5, 87.2)
- moved C1 526.6 mm to (44.6, 129.1)
- moved C2 526.6 mm to (25.3, 132.9)
- moved C3 526.6 mm to (41.8, 123.5)
- moved C4 526.6 mm to (35.8, 104.2)
- moved C5 526.6 mm to (35.8, 106.7)
- moved D1 526.6 mm to (25.5, 121.0)
- moved D10 526.6 mm to (34.4, 124.0)
- moved D11 526.6 mm to (34.4, 127.0)
- moved D12 526.6 mm to (34.4, 130.1)
- moved D13 526.6 mm to (39.5, 129.3)
- moved D2 526.6 mm to (25.5, 124.0)
- moved D3 526.6 mm to (25.5, 127.0)
- moved D4 526.6 mm to (25.5, 130.1)
- moved D5 526.6 mm to (30.0, 121.0)
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Connections:
- net /BLU_ON renamed //CMD

Commit message: pcb
Parts:
- moved C6 134.9 mm to (66.4, 123.8)
- moved U2 134.9 mm to (66.7, 120.1)
Changed lines of the file:
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@@
   (net 33 "/{slash}CMD")
   (footprint "Capacitor_SMD:C_0805_2012Metric" (layer "F.Cu")
-    (at 1.725 5.455)
+    (at 66.36 123.825)
     (descr "Capacitor SMD 0805 (2012 Metric), square (rectangular) end terminal, IPC_7351 nominal, (Body size source: IPC-SM-782 page 76, https://www.pcb-3d.com/wordpress/wp-content/uploads/ipc-sm-782a_amendment_1_and_2.pdf, https://docs.google.com/spreadsheets/d/1BsfQQcO9C6DZCsRaXUlFlo91Tg2WpOkGARC1WS5S8t0/edit?usp=sharing), generated with kicad-footprint-generator")
     (tags "capacitor")
@@
   )
   (footprint "Package_TO_SOT_SMD:SOT-23-5" (layer "F.Cu")
-    (at 2.075 1.725)
+    (at 66.71 120.095)
     (descr "SOT, 5 Pin (https://www.jedec.org/sites/default/files/docs/Mo-178c.PDF variant AA), generated with kicad-footprint-generator ipc_gullwing_generator.py")
     (tags "SOT TO_SOT_SMD")

Commit message: trims
Parts:
- moved R8 45.2 mm to (56.1, 109.2)
Connections:
- net /CV1 renamed /CCV1
- net /CV2 renamed /CCV2
- net Net-(D1-K) renamed /V1 1-2
- net Net-(D10-A) renamed /V2 2-3
- net Net-(D11-A) renamed /B1 2-3
- net Net-(D12-A) renamed /B2 2-3
- net Net-(D2-K) renamed /V2 1-2
- net Net-(D3-K) renamed /B1 1-2
- net Net-(D4-K) renamed /B2 1-2
- net Net-(D5-K) renamed /V1 2-3
Changed lines of the file:
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@@
   (net 5 "/THR")
   (net 6 "/9V")
-  (net 7 "Net-(D1-K)")
-  (net 8 "Net-(D2-K)")
-  (net 9 "Net-(D3-K)")
-  (net 10 "Net-(D4-K)")
-  (net 11 "Net-(D5-K)")
-  (net 12 "Net-(D10-A)")
-  (net 13 "Net-(D11-A)")
-  (net 14 "Net-(D12-A)")
-  (net 15 "/CV1")
-  (net 16 "/CV2")
+  (net 7 "/V1 1-2")
+  (net 8 "/V2 1-2")
+  (net 9 "/B1 1-2")
+  (net 10 "/B2 1-2")
+  (net 11 "/V1 2-3")
+  (net 12 "/V2 2-3")
+  (net 13 "/B1 2-3")
+  (net 14 "/B2 2-3")
+  (net 15 "/CCV1")
+  (net 16 "/CCV2")
   (net 17 "/CB1")
   (net 18 "/CB2")
@@
       (stroke (width 0.1) (type solid)) (layer "F.Fab"))
     (pad "1" smd roundrect (at -0.9375 0) (size 0.975 1.4) (layers "F.Cu" "F.Paste" "F.Mask") (roundrect_rratio 0.25)
-      (net 13 "Net-(D11-A)") (pinfunction "K") (pintype "passive"))
+      (net 13 "/B1 2-3") (pinfunction "K") (pintype "passive"))
     (pad "2" smd roundrect (at 0.9375 0) (size 0.975 1.4) (layers "F.Cu" "F.Paste" "F.Mask") (roundrect_rratio 0.25)
-      (net 9 "Net-(D3-K)") (pinfunction "A") (pintype "passive"))
+      (net 9 "/B1 1-2") (pinfunction "A") (pintype "passive"))
     (model "${KICAD6_3DMODEL_DIR}/LED_SMD.3dshapes/LED_0805_2012Metric.wrl"
       (offset (xyz 0 0 0))
@@
       (stroke (width 0.1) (type solid)) (layer "F.Fab"))
     (pad "1" smd roundrect (at -0.9375 0) (size 0.975 1.4) (layers "F.Cu" "F.Paste" "F.Mask") (roundrect_rratio 0.25)
-      (net 15 "/CV1") (pinfunction "K") (pintype "passive"))
+      (net 15 "/CCV1") (pinfunction "K") (pintype "passive"))
     (pad "2" smd roundrect (at 0.9375 0) (size 0.975 1.4) (layers "F.Cu" "F.Paste" "F.Mask") (roundrect_rratio 0.25)
-      (net 11 "Net-(D5-K)") (pinfunction "A") (pintype "passive"))
+      (net 11 "/V1 2-3") (pinfunction "A") (pintype "passive"))
     (model "${KICAD6_3DMODEL_DIR}/LED_SMD.3dshapes/LED_0805_2012Metric.wrl"
       (offset (xyz 0 0 0))
@@
       (stroke (width 0.1) (type solid)) (layer "F.Fab"))
     (pad "1" smd roundrect (at -0.9375 0) (size 0.975 1.4) (layers "F.Cu" "F.Paste" "F.Mask") (roundrect_rratio 0.25)
-      (net 10 "Net-(D4-K)") (pinfunction "K") (pintype "passive"))
+      (net 10 "/B2 1-2") (pinfunction "K") (pintype "passive"))
     (pad "2" smd roundrect (at 0.9375 0) (size 0.975 1.4) (layers "F.Cu" "F.Paste" "F.Mask") (roundrect_rratio 0.25)
       (net 6 "/9V") (pinfunction "A") (pintype "passive"))
@@
       (net 18 "/CB2") (pinfunction "K") (pintype "passive"))
     (pad "2" smd roundrect (at 0.9375 0) (size 0.975 1.4) (layers "F.Cu" "F.Paste" "F.Mask") (roundrect_rratio 0.25)
-      (net 14 "Net-(D12-A)") (pinfunction "A") (pintype "passive"))
+      (net 14 "/B2 2-3") (pinfunction "A") (pintype "passive"))
     (model "${KICAD6_3DMODEL_DIR}/LED_SMD.3dshapes/LED_0805_2012Metric.wrl"
       (offset (xyz 0 0 0))
@@
       (stroke (width 0.1) (type solid)) (layer "F.Fab"))
     (pad "1" smd roundrect (at -0.9375 0) (size 0.975 1.4) (layers "F.Cu" "F.Paste" "F.Mask") (roundrect_rratio 0.25)
-      (net 14 "Net-(D12-A)") (pinfunction "K") (pintype "passive"))
+      (net 14 "/B2 2-3") (pinfunction "K") (pintype "passive"))
     (pad "2" smd roundrect (at 0.9375 0) (size 0.975 1.4) (layers "F.Cu" "F.Paste" "F.Mask") (roundrect_rratio 0.25)
-      (net 10 "Net-(D4-K)") (pinfunction "A") (pintype "passive"))
+      (net 10 "/B2 1-2") (pinfunction "A") (pintype "passive"))
     (model "${KICAD6_3DMODEL_DIR}/LED_SMD.3dshapes/LED_0805_2012Metric.wrl"
       (offset (xyz 0 0 0))
@@
       (net 17 "/CB1") (pinfunction "K") (pintype "passive"))
     (pad "2" smd roundrect (at 0.9375 0) (size 0.975 1.4) (layers "F.Cu" "F.Paste" "F.Mask") (roundrect_rratio 0.25)
-      (net 13 "Net-(D11-A)") (pinfunction "A") (pintype "passive"))
+      (net 13 "/B1 2-3") (pinfunction "A") (pintype "passive"))
     (model "${KICAD6_3DMODEL_DIR}/LED_SMD.3dshapes/LED_0805_2012Metric.wrl"
       (offset (xyz 0 0 0))
@@
   )
   (footprint "PVG5A202C03R00:TRIM_PVG5A202C03R00" (layer "F.Cu")
-    (at 20.25 136.72)
+    (at 56.06 109.2)
     (property "Purpose" "TB2")
     (property "Sheetfile" "tannenbaum.kicad_sch")
@@
       (stroke (width 0.1) (type solid)) (layer "F.Fab"))
     (pad "1" smd roundrect (at -0.9375 0) (size 0.975 1.4) (layers "F.Cu" "F.Paste" "F.Mask") (roundrect_rratio 0.25)
-      (net 8 "Net-(D2-K)") (pinfunction "K") (pintype "passive"))
+      (net 8 "/V2 1-2") (pinfunction "K") (pintype "passive"))
     (pad "2" smd roundrect (at 0.9375 0) (size 0.975 1.4) (layers "F.Cu" "F.Paste" "F.Mask") (roundrect_rratio 0.25)
       (net 6 "/9V") (pinfunction "A") (pintype "passive"))
@@
       (stroke (width 0.1) (type solid)) (layer "F.Fab"))
     (pad "1" smd roundrect (at -0.9375 0) (size 0.975 1.4) (layers "F.Cu" "F.Paste" "F.Mask") (roundrect_rratio 0.25)
-      (net 11 "Net-(D5-K)") (pinfunction "K") (pintype "passive"))
+      (net 11 "/V1 2-3") (pinfunction "K") (pintype "passive"))
     (pad "2" smd roundrect (at 0.9375 0) (size 0.975 1.4) (layers "F.Cu" "F.Paste" "F.Mask") (roundrect_rratio 0.25)
-      (net 7 "Net-(D1-K)") (pinfunction "A") (pintype "passive"))
+      (net 7 "/V1 1-2") (pinfunction "A") (pintype "passive"))
     (model "${KICAD6_3DMODEL_DIR}/LED_SMD.3dshapes/LED_0805_2012Metric.wrl"
       (offset (xyz 0 0 0))
@@
       (stroke (width 0.1) (type solid)) (layer "F.Fab"))
     (pad "1" smd roundrect (at -0.9375 0) (size 0.975 1.4) (layers "F.Cu" "F.Paste" "F.Mask") (roundrect_rratio 0.25)
-      (net 12 "Net-(D10-A)") (pinfunction "K") (pintype "passive"))
+      (net 12 "/V2 2-3") (pinfunction "K") (pintype "passive"))
     (pad "2" smd roundrect (at 0.9375 0) (size 0.975 1.4) (layers "F.Cu" "F.Paste" "F.Mask") (roundrect_rratio 0.25)
-      (net 8 "Net-(D2-K)") (pinfunction "A") (pintype "passive"))
+      (net 8 "/V2 1-2") (pinfunction "A") (pintype "passive"))
     (model "${KICAD6_3DMODEL_DIR}/LED_SMD.3dshapes/LED_0805_2012Metric.wrl"
       (offset (xyz 0 0 0))
@@
       (stroke (width 0.1) (type solid)) (layer "F.Fab"))
     (pad "1" smd roundrect (at -0.9375 0) (size 0.975 1.4) (layers "F.Cu" "F.Paste" "F.Mask") (roundrect_rratio 0.25)
-      (net 16 "/CV2") (pinfunction "K") (pintype "passive"))
+      (net 16 "/CCV2") (pinfunction "K") (pintype "passive"))
     (pad "2" smd roundrect (at 0.9375 0) (size 0.975 1.4) (layers "F.Cu" "F.Paste" "F.Mask") (roundrect_rratio 0.25)
-      (net 12 "Net-(D10-A)") (pinfunction "A") (pintype "passive"))
+      (net 12 "/V2 2-3") (pinfunction "A") (pintype "passive"))
     (model "${KICAD6_3DMODEL_DIR}/LED_SMD.3dshapes/LED_0805_2012Metric.wrl"
       (offset (xyz 0 0 0))
@@
       (net 20 "Net-(Q1-E)") (pinfunction "E") (pintype "passive") (solder_mask_margin 0.07))
     (pad "3" smd rect (at 1.05 0) (size 1.3 0.6) (layers "F.Cu" "F.Paste" "F.Mask")
-      (net 15 "/CV1") (pinfunction "C") (pintype "passive") (solder_mask_margin 0.07))
+      (net 15 "/CCV1") (pinfunction "C") (pintype "passive") (solder_mask_margin 0.07))
   )
   (footprint "digikey-footprints:SOT-23-3" (layer "F.Cu")
@@
       (net 22 "Net-(Q2-E)") (pinfunction "E") (pintype "passive") (solder_mask_margin 0.07))
     (pad "3" smd rect (at 1.05 0) (size 1.3 0.6) (layers "F.Cu" "F.Paste" "F.Mask")
-      (net 16 "/CV2") (pinfunction "C") (pintype "passive") (solder_mask_margin 0.07))
+      (net 16 "/CCV2") (pinfunction "C") (pintype "passive") (solder_mask_margin 0.07))
   )
   (footprint "PVG5A202C03R00:TRIM_PVG5A202C03R00" (layer "F.Cu")
@@
       (stroke (width 0.1) (type solid)) (layer "F.Fab"))
     (pad "1" smd roundrect (at -0.9375 0) (size 0.975 1.4) (layers "F.Cu" "F.Paste" "F.Mask") (roundrect_rratio 0.25)
-      (net 9 "Net-(D3-K)") (pinfunction "K") (pintype "passive"))
+      (net 9 "/B1 1-2") (pinfunction "K") (pintype "passive"))
     (pad "2" smd roundrect (at 0.9375 0) (size 0.975 1.4) (layers "F.Cu" "F.Paste" "F.Mask") (roundrect_rratio 0.25)
       (net 6 "/9V") (pinfunction "A") (pintype "passive"))
@@
       (stroke (width 0.1) (type solid)) (layer "F.Fab"))
     (pad "1" smd roundrect (at -0.9375 0) (size 0.975 1.4) (layers "F.Cu" "F.Paste" "F.Mask") (roundrect_rratio 0.25)
-      (net 7 "Net-(D1-K)") (pinfunction "K") (pintype "passive"))
+      (net 7 "/V1 1-2") (pinfunction "K") (pintype "passive"))
     (pad "2" smd roundrect (at 0.9375 0) (size 0.975 1.4) (layers "F.Cu" "F.Paste" "F.Mask") (roundrect_rratio 0.25)
       (net 6 "/9V") (pinfunction "A") (pintype "passive"))

Commit message: pcb
Parts:
- moved BT1 187.7 mm to (224.8, 34.9)
- moved D9 50.9 mm to (70.2, 84.7)
- moved D1 50.9 mm to (61.3, 84.7)
- moved D10 50.9 mm to (70.2, 87.8)
- moved D11 50.9 mm to (70.2, 90.8)
- moved D5 50.9 mm to (65.7, 84.7)
- moved D2 50.9 mm to (61.3, 87.8)
- moved D3 50.9 mm to (61.3, 90.8)
- moved D6 50.9 mm to (65.7, 87.8)
- moved D7 50.9 mm to (65.7, 90.8)
Other:
- board outline added: 228 x 153 mm
Changed lines of the file:
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@@
   )
   (footprint "BH9VW:BAT_BH9VW_SMD" (layer "F.Cu")
-    (at 44.53 87.17)
+    (at 224.79 34.925)
     (property "Check_prices" "https://www.snapeda.com/parts/BH9VW/MPD+%2528Memory+Protection+Devices%2529/view-part/?ref=eda")
     (property "Description" "\nBattery Holder (Open) 9V 1 Cell Wire Leads - 6 (152.4mm)\n")
@@
   )
   (footprint "LED_SMD:LED_0805_2012Metric" (layer "F.Cu")
-    (at 29.965 127.045)
+    (at 65.7325 90.805)
     (descr "LED SMD 0805 (2012 Metric), square (rectangular) end terminal, IPC_7351 nominal, (Body size source: https://docs.google.com/spreadsheets/d/1BsfQQcO9C6DZCsRaXUlFlo91Tg2WpOkGARC1WS5S8t0/edit?usp=sharing), generated with kicad-footprint-generator")
     (tags "LED")
@@
   )
   (footprint "LED_SMD:LED_0805_2012Metric" (layer "F.Cu")
-    (at 34.415 120.965)
+    (at 70.1825 84.725)
     (descr "LED SMD 0805 (2012 Metric), square (rectangular) end terminal, IPC_7351 nominal, (Body size source: https://docs.google.com/spreadsheets/d/1BsfQQcO9C6DZCsRaXUlFlo91Tg2WpOkGARC1WS5S8t0/edit?usp=sharing), generated with kicad-footprint-generator")
     (tags "LED")
@@
     (property "ki_keywords" "LED diode")
     (attr smd)
-    (fp_text reference "D4" (at 0 -1.65) (layer "F.SilkS")
+    (fp_text reference "D4" (at 35.7675 -37.89) (layer "F.SilkS")
         (effects (font (size 1 1) (thickness 0.15)))
     )
@@
         (effects (font (size 1 1) (thickness 0.15)))
     )
-    (fp_text user "${REFERENCE}" (at 0 0) (layer "F.Fab")
+    (fp_text user "${REFERENCE}" (at 35.7675 -36.24) (layer "F.Fab")
         (effects (font (size 0.5 0.5) (thickness 0.08)))
     )
@@
     (property "ki_keywords" "LED diode")
     (attr smd)
-    (fp_text reference "D12" (at 0 -1.65) (layer "F.SilkS")
+    (fp_text reference "D12" (at 35.7675 -37.89) (layer "F.SilkS")
         (effects (font (size 1 1) (thickness 0.15)))
     )
@@
         (effects (font (size 1 1) (thickness 0.15)))
     )
-    (fp_text user "${REFERENCE}" (at 0 0) (layer "F.Fab")
+    (fp_text user "${REFERENCE}" (at 35.7675 -36.24) (layer "F.Fab")
         (effects (font (size 0.5 0.5) (thickness 0.08)))
     )
@@
     (property "ki_keywords" "LED diode")
     (attr smd)
-    (fp_text reference "D8" (at 0 -1.65) (layer "F.SilkS")
+    (fp_text reference "D8" (at 35.7675 -37.89) (layer "F.SilkS")
         (effects (font (size 1 1) (thickness 0.15)))
     )
@@
         (effects (font (size 1 1) (thickness 0.15)))
     )
-    (fp_text user "${REFERENCE}" (at 0 0) (layer "F.Fab")
+    (fp_text user "${REFERENCE}" (at 35.7675 -36.24) (layer "F.Fab")
         (effects (font (size 0.5 0.5) (thickness 0.08)))
     )
@@
   )
   (footprint "LED_SMD:LED_0805_2012Metric" (layer "F.Cu")
-    (at 34.415 127.045)
+    (at 70.1825 90.805)
     (descr "LED SMD 0805 (2012 Metric), square (rectangular) end terminal, IPC_7351 nominal, (Body size source: https://docs.google.com/spreadsheets/d/1BsfQQcO9C6DZCsRaXUlFlo91Tg2WpOkGARC1WS5S8t0/edit?usp=sharing), generated with kicad-footprint-generator")
     (tags "LED")
@@
   )
   (footprint "LED_SMD:LED_0805_2012Metric" (layer "F.Cu")
-    (at 25.515 124.005)
+    (at 61.2825 87.765)
     (descr "LED SMD 0805 (2012 Metric), square (rectangular) end terminal, IPC_7351 nominal, (Body size source: https://docs.google.com/spreadsheets/d/1BsfQQcO9C6DZCsRaXUlFlo91Tg2WpOkGARC1WS5S8t0/edit?usp=sharing), generated with kicad-footprint-generator")
     (tags "LED")
@@
   )
   (footprint "LED_SMD:LED_0805_2012Metric" (layer "F.Cu")
-    (at 29.965 120.965)
+    (at 65.7325 84.725)
     (descr "LED SMD 0805 (2012 Metric), square (rectangular) end terminal, IPC_7351 nominal, (Body size source: https://docs.google.com/spreadsheets/d/1BsfQQcO9C6DZCsRaXUlFlo91Tg2WpOkGARC1WS5S8t0/edit?usp=sharing), generated with kicad-footprint-generator")
     (tags "LED")
@@
   )
   (footprint "LED_SMD:LED_0805_2012Metric" (layer "F.Cu")
-    (at 29.965 124.005)
+    (at 65.7325 87.765)
     (descr "LED SMD 0805 (2012 Metric), square (rectangular) end terminal, IPC_7351 nominal, (Body size source: https://docs.google.com/spreadsheets/d/1BsfQQcO9C6DZCsRaXUlFlo91Tg2WpOkGARC1WS5S8t0/edit?usp=sharing), generated with kicad-footprint-generator")
     (tags "LED")
@@
   )
   (footprint "LED_SMD:LED_0805_2012Metric" (layer "F.Cu")
-    (at 34.415 124.005)
+    (at 70.1825 87.765)
     (descr "LED SMD 0805 (2012 Metric), square (rectangular) end terminal, IPC_7351 nominal, (Body size source: https://docs.google.com/spreadsheets/d/1BsfQQcO9C6DZCsRaXUlFlo91Tg2WpOkGARC1WS5S8t0/edit?usp=sharing), generated with kicad-footprint-generator")
     (tags "LED")
@@
         (effects (font (size 1 1) (thickness 0.15)))
     )
-    (fp_text value "R_Trim" (at 9.144 3.683) (layer "F.Fab")
+    (fp_text value "R_Trim" (at 44.9115 -32.557) (layer "F.Fab")
         (effects (font (size 1 1) (thickness 0.15)))
     )
@@
   )
   (footprint "LED_SMD:LED_0805_2012Metric" (layer "F.Cu")
-    (at 25.515 127.045)
+    (at 61.2825 90.805)
     (descr "LED SMD 0805 (2012 Metric), square (rectangular) end terminal, IPC_7351 nominal, (Body size source: https://docs.google.com/spreadsheets/d/1BsfQQcO9C6DZCsRaXUlFlo91Tg2WpOkGARC1WS5S8t0/edit?usp=sharing), generated with kicad-footprint-generator")
     (tags "LED")
@@
         (effects (font (size 1 1) (thickness 0.15)))
     )
-    (fp_text value "R_Trim" (at 9.144 3.683) (layer "F.Fab")
+    (fp_text value "R_Trim" (at 44.9115 -32.557) (layer "F.Fab")
         (effects (font (size 1 1) (thickness 0.15)))
     )
@@
   )
   (footprint "LED_SMD:LED_0805_2012Metric" (layer "F.Cu")
-    (at 25.515 120.965)
+    (at 61.2825 84.725)
     (descr "LED SMD 0805 (2012 Metric), square (rectangular) end terminal, IPC_7351 nominal, (Body size source: https://docs.google.com/spreadsheets/d/1BsfQQcO9C6DZCsRaXUlFlo91Tg2WpOkGARC1WS5S8t0/edit?usp=sharing), generated with kicad-footprint-generator")
     (tags "LED")
@@
       (net 3 "/3V3") (pinfunction "VOUT") (pintype "passive"))
   )
+  (gr_poly
+    (pts
+      (xy 37.465 64.135)
+      (xy 64.135 67.31)
+      (xy 63.5 16.51)
+      (xy 114.935 73.66)
+      (xy 114.935 36.195)
+      (xy 167.005 81.28)
+      (xy 167.005 56.515)
+      (xy 216.535 88.9)
+      (xy 216.535 76.835)
+      (xy 264.16 95.25)
+      (xy 216.535 113.03)
+      (xy 216.535 101.6)
+      (xy 167.005 131.445)
+      (xy 167.005 107.95)
+      (xy 114.935 149.86)
+      (xy 114.935 114.935)
+      (xy 64.135 169.545)
+      (xy 64.77 120.65)
+      (xy 36.195 125.095)
+      (xy 36.195 63.5)
+    )
+    (stroke (width 0.1) (type solid)) (fill none) (layer "Edge.Cuts"))
 )
