File: tannenbaum.kicad_pcb (KiCad board)
At the start: 2 copper layers, 228 x 153 mm, 42 parts, among them Q1 MMBT3904-7-F, Q2 MMBT3904-7-F, Q3 MMBT3904-7-F, Q4 MMBT3904-7-F, Q5 2N7002, Q6 BSS84, SW1 SW_SPDT, U1 ICM7555xB, U2 LP2985-3.3

Commit message: gerber
Parts:
- added D14: LED, LED_SMD:LED_0805_2012Metric_LW, F.Cu at (123.8, 106.0)
- added D15: LED, LED_SMD:LED_0805_2012Metric_LW, F.Cu at (146.7, 112.4)
- added D16: LED, LED_SMD:LED_0805_2012Metric_LW, F.Cu at (148.6, 76.2)
- added D17: LED, LED_SMD:LED_0805_2012Metric_LW, F.Cu at (174.6, 111.1)
- added D18: LED, LED_SMD:LED_0805_2012Metric_LW, F.Cu at (187.3, 76.5)
- added D19: LED, LED_SMD:LED_0805_2012Metric_LW, F.Cu at (220.3, 101.0)
- added Q7: MMBT3904-7-F, digikey-footprints:SOT-23-3, B.Cu at (208.7, 100.7)
- added Q8: BSS84, digikey-footprints:SOT-23-3, B.Cu at (62.2, 73.0)
- added R14: R_Trim, Potentiometer_SMD:Potentiometer_Bourns_TC33X_Vertical, B.Cu at (137.3, 69.5)
- added R15: 1K2, Resistor_SMD:R_0603_1608Metric, B.Cu at (208.7, 96.5)
- added R16: R_Trim, Potentiometer_SMD:Potentiometer_Bourns_TC33X_Vertical, B.Cu at (213.5, 96.9)
- added R17: 0R, Resistor_SMD:R_0805_2012Metric, B.Cu at (68.6, 70.8)
- BT1, C3, C4, Q1, Q2, Q3, R10, R4, SW1, U1, U2: moved to B.Cu
- C1: value 100n -> 100p; footprint Capacitor_SMD:C_0805_2012Metric -> Capacitor_SMD:C_0603_1608Metric; moved to B.Cu
- C2: value 100p -> 100n; footprint Capacitor_SMD:C_0603_1608Metric -> Capacitor_SMD:C_0805_2012Metric; moved to B.Cu
- C5: value 1u -> 10n; footprint Capacitor_SMD:C_0603_1608Metric -> Capacitor_SMD:C_0805_2012Metric; moved to B.Cu
- C6: value 10n -> 1u; footprint Capacitor_SMD:C_0805_2012Metric -> Capacitor_SMD:C_0603_1608Metric; moved to B.Cu
- D1: value LED -> 1N4148W; footprint LED_SMD:LED_0805_2012Metric_LW -> Diode_SMD:D_SOD-123; moved to B.Cu
- D13: value 1N4148W -> LED; footprint Diode_SMD:D_SOD-123 -> LED_SMD:LED_0805_2012Metric_LW
- Q4: value MMBT3904-7-F -> 2N7002; moved to B.Cu
- Q5: value 2N7002 -> MMBT3904-7-F; moved to B.Cu
- Q6: value BSS84 -> MMBT3904-7-F; moved to B.Cu
- R1, R2, R3: value 1K2 -> 100k; footprint Resistor_SMD:R_0603_1608Metric -> Resistor_SMD:R_0805_2012Metric; moved to B.Cu
- R11: value 100k -> 1K2; footprint Resistor_SMD:R_0805_2012Metric -> Resistor_SMD:R_0603_1608Metric; moved to B.Cu
- R12, R9: value 100k -> R_Trim; footprint Resistor_SMD:R_0805_2012Metric -> Potentiometer_SMD:Potentiometer_Bourns_TC33X_Vertical; moved to B.Cu
- R13: value 0R -> 1K2; footprint Resistor_SMD:R_0805_2012Metric -> Resistor_SMD:R_0603_1608Metric; moved to B.Cu
- R5, R7: footprint PVG5A202C03R00:TRIM_PVG5A202C03R00_TWO -> Potentiometer_SMD:Potentiometer_Bourns_TC33X_Vertical; moved to B.Cu
- R6, R8: value R_Trim -> 1K2; footprint PVG5A202C03R00:TRIM_PVG5A202C03R00_TWO -> Resistor_SMD:R_0603_1608Metric; moved to B.Cu
- moved BT1 171.4 mm to (63.7, 93.3)
- moved R4 151.9 mm to (165.7, 85.1), turned to 180 degrees
- moved D8 151.6 mm to (227.3, 92.7), turned to 90 degrees
- moved Q1 149.1 mm to (171.4, 85.7)
- moved R5 143.4 mm to (160.1, 86.0), turned to 180 degrees
- moved R9 128.8 mm to (153.0, 92.1), turned to 90 degrees
- moved Q3 126.0 mm to (159.4, 96.7)
- moved R13 111.0 mm to (143.5, 69.2), turned to 180 degrees
- moved D9 110.6 mm to (185.4, 104.8), turned to -90 degrees
- moved Q6 107.9 mm to (143.2, 73.4), turned to -90 degrees
- moved D4 106.6 mm to (178.4, 84.2), turned to 90 degrees
- moved R7 104.9 mm to (125.1, 134.6), turned to -90 degrees
- moved R8 103.2 mm to (157.9, 92.7), turned to 180 degrees
- moved R6 101.4 mm to (121.3, 132.1), turned to -90 degrees
- moved Q2 94.8 mm to (124.5, 128.3), turned to 90 degrees
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Connections:
- C1 pad 1: GND -> Net-(U1-CV)
- C1 pad 2: /3V3 -> GND
- C2 pad 1: Net-(U1-CV) -> GND
- C2 pad 2: GND -> /3V3
- C5 pad 1: /3V3 -> Net-(U2-BP)
- C6 pad 1: Net-(U2-BP) -> /3V3
- D1 pad 1: /V1 1-2 -> /THR
- D1 pad 2: /9V -> /DSC
- D10 pad 1: /CCV2 -> /CCV3
- D10 pad 2: /V2 2-3 -> /V3 2-3
- D11 pad 1: /CB1 -> /B1 1-2
- D11 pad 2: /B1 2-3 -> /9V
- D12 pad 1: /CB2 -> /B1 2-3
- D12 pad 2: /B2 2-3 -> /B1 1-2
- D13 pad 1: /THR -> /CB1
- D13 pad 2: /DSC -> /B1 2-3
- D2 pad 1: /V2 1-2 -> /V1 1-2
- D3 pad 1: /B1 1-2 -> /V1 2-3
- D3 pad 2: /9V -> /V1 1-2
- D4 pad 1: /B2 1-2 -> /CCV1
- D4 pad 2: /9V -> /V1 2-3
- D5 pad 1: /V1 2-3 -> /V2 1-2
- D5 pad 2: /V1 1-2 -> /9V
- D7 pad 1: /B1 2-3 -> /CCV2
- D7 pad 2: /B1 1-2 -> /V2 2-3
- D8 pad 1: /B2 2-3 -> /V3 1-2
- D8 pad 2: /B2 1-2 -> /9V
- D9 pad 1: /CCV1 -> /V3 2-3
- D9 pad 2: /V1 2-3 -> /V3 1-2
- Q3 pad 1: //CMD -> /CMD
- Q3 pad 3: /CB1 -> /CCV3
- Q4 pad 1: //CMD -> /CMD
- Q4 pad 2: Net-(Q4-E) -> GND
- Q4 pad 3: /CB2 -> //CMD
- Q5 pad 1: /CMD -> //CMD
- Q5 pad 2: GND -> Net-(Q5-E)
- Q5 pad 3: //CMD -> /CB1
- Q6 pad 1: GND -> //CMD
- Q6 pad 2: Net-(Q6-D) -> Net-(Q6-E)
- Q6 pad 3: /9V -> /CB2
- R1 pad 1: Net-(Q2-E) -> /CMD
- R1 pad 2: Net-(R1-Pad2) -> Net-(U1-Q)
- R10 pad 1: /DSC -> /3V3
- R10 pad 2: /THR -> //CMD
- R11 pad 1: /DSC -> Net-(Q5-E)
- R11 pad 2: /3V3 -> Net-(R11-Pad2)
- R12 pad 1: /CMD -> Net-(R11-Pad2)
- R12 pad 2: Net-(U1-Q) -> GND
- R13 pad 1: Net-(Q6-D) -> Net-(Q6-E)
- R13 pad 2: /9V -> Net-(R13-Pad2)
- R2 pad 1: Net-(Q3-E) -> /DSC
- R2 pad 2: Net-(R2-Pad2) -> /3V3
- R3 pad 1: Net-(Q4-E) -> /DSC
- R3 pad 2: Net-(R3-Pad2) -> /THR
- R6 pad 1: Net-(R1-Pad2) -> Net-(Q2-E)
- R6 pad 2: GND -> Net-(R6-Pad2)
- R7 pad 1: Net-(R2-Pad2) -> Net-(R6-Pad2)
- R8 pad 1: Net-(R3-Pad2) -> Net-(Q3-E)
- R8 pad 2: GND -> Net-(R8-Pad2)
- R9 pad 1: /3V3 -> Net-(R8-Pad2)
- R9 pad 2: //CMD -> GND
- SW1 pad 3: Net-(Q6-D) -> Net-(Q8-D)
Routing:
- net /9V: track 0.00 -> 388.0 mm, vias 0 -> 6
- net //CMD: track 0.00 -> 356.0 mm, vias 0 -> 2
- net /CMD: track 0.00 -> 164.0 mm, vias 0 -> 2
- net /V1 1-2: track 0.00 -> 84.8 mm, vias 0 -> 2
- net /B3 2-3: track 0.00 -> 63.3 mm, vias 0 -> 2
- net /B3 1-2: track 0.00 -> 56.4 mm, vias 0 -> 2
- net /V1 2-3: track 0.00 -> 54.7 mm, vias 0 -> 2
- net /V2 1-2: track 0.00 -> 51.8 mm, vias 0 -> 2
- net /V3 1-2: track 0.00 -> 47.2 mm, vias 0 -> 2
- net /THR: track 0.00 -> 42.6 mm
- net /V2 2-3: track 0.00 -> 40.7 mm, vias 0 -> 2
- net /B2 2-3: track 0.00 -> 35.1 mm, vias 0 -> 2
- net /B1 1-2: track 0.00 -> 30.1 mm, vias 0 -> 2
- net /B2 1-2: track 0.00 -> 26.9 mm, vias 0 -> 2
- net /PSU/VBat: track 0.00 -> 25.8 mm
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- added copper zone on B.Cu, net GND
- added copper zone on F.Cu, net GND
Other:
- outline, holes or cut-outs redrawn
