File: tannenbaum.kicad_pcb (KiCad board)
At the start: 2 copper layers, 228 x 153 mm, 54 parts, among them Q1 MMBT3904-7-F, Q2 MMBT3904-7-F, Q3 MMBT3904-7-F, Q4 2N7002, Q5 MMBT3904-7-F, Q6 MMBT3904-7-F, Q7 MMBT3904-7-F, Q8 BSS84, SW1 SW_SPDT, U1 ICM7555xB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

Commit message: finish
Other:
- board text added: "JLCJLCJLCJLC"
Changed lines of the file:
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@@
     )
     (stroke (width 0.1) (type solid)) (fill none) (layer "Edge.Cuts"))
+  (gr_text "JLCJLCJLCJLC" (at 68.58 93.98) (layer "B.SilkS")
+    (effects (font (size 1 1) (thickness 0.15)) (justify left bottom mirror))
+  )
   (segment (start 95.9825 87.17) (end 88.695 87.17) (width 0.25) (layer "B.Cu") (net 1))
   (segment (start 88.695 87.17) (end 75.605 74.08) (width 0.25) (layer "B.Cu") (net 1))
